File: KiCad/KiCad-DimSumRobot.kicad_sch (KiCad schematic)
At the start: 13 parts, among them J1 SHT40, J2 Ultrasonic Radar, J3 JST PH2.0, J4 MT3608, M1 Left Motor, M2 Right Motor, SW1 ON/OFF Switch, U1 XIAO-ESP32-S3-SMD, U2 TB6612FNG, U3 MPU-6050

Commit message: Add files via upload
Remapping GND to correct electromagnetic interference which was the root of my MPU not working properly
Parts:
- added C3: 0.1uf, symbol Device:C
- added C4: 100uf 25V, symbol Device:C_Polarized
- added R1, R2: 4.7K, symbol Device:R
- added U4: ADS1115, Package_SO:TSSOP-10_3x3mm_P0.5mm, symbol Analog_ADC:ADS1115IDGS
Connections:
- net at J4.1 (VIN+), SW1.1 (A), U1.23 (BAT+): now also R1.2
- net at BT1.2 (-), J3.2 (Pin_2), J4.2 (VIN-)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: now also U2.3 (PGND1), U2.4 (PGND1), R2.2; no longer J1.1 (GND), J2.1 (GND), U1.13 (GND), U3.18 (GND)
- net at J1.2 (VCC), J2.2 (VCC), U1.12 (3V3_OUT)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: now also C3.1, C4.1, U4.8 (VDD)
- net at J1.3 (SDA), U1.5 (D4), U3.24 (SDA): now also U4.9 (SDA)
- net at J1.4 (SCL), U1.6 (D5), U3.23 (SCL): now also U4.10 (SCL)
- new net: C3.2, C4.2, J1.1 (GND), J2.1 (GND), U1.13 (GND), U3.18 (GND), U4.3 (GND)
- new net: R1.1, R2.1, U4.4 (AIN0)
Other:
- moved on the sheet: M1, M2, U1
